File: eagle/Slave/v1.brd (EAGLE design)
At the start: 99.2 x 69.3 mm, 54 parts, among them CON1 SPI, J1 RJ12, J2 RJ12, J3 RJ12, Q1 BSP75, Q10 BSP75, Q11 BSP75, Q12 BSP75, Q13 BSP75, Q2 BSP75, Q3 BSP75, Q4 BSP75, Q5 BSP75, Q6 BSP75, Q7 BSP75, Q8 BSP75, Q9 BSP75, X3 16MHz, X4 MINI-USB

Commit message: Update eagle
Parts:
- removed LED10: GREEN, adafruit:CHIP-LED0805
- removed Q13, Q3, Q5, Q6: BSP75, infineon:PG-SOT-223
- removed RL3: 1K, rcl:R0805
- removed U$6: KPJX-4S-S, lpatiny:KPJX-4S-S
- added C25, C26: 1nF, freetronics-master-v1:0805
- added C27: 100n, freetronics-master-v1:0805
- added C28, C31, C32, C33: 100nF, freetronics-master-v1:0805
- added C29, C34, C35: 220n, freetronics-master-v1:0805
- added C30: 100nF, freetronics-master-v1:0603
- added C47: 100uF 50V, freetronics-original:PANASONIC_E
- added IC4: DRV8811, eje-components:HTSSOP28
- added JP3: (no value), jumper:JP4
- added R1: 3k3, freetronics-master-v1:0805
- added R2, R34, R35, R36, R5, R6, R7: 10k, freetronics-master-v1:0805
- added R25, R27: 47K, freetronics-master-v1:0805
- added R26, R38: 0.2R 1W, rcl:R2010
- added R28: 0R, freetronics-master-v1:0805
- added R37: 4K7, freetronics-master-v1:0805
- added SJ7: MS1, freetronics-luke:SJ
- added SJ8: MS0, freetronics-luke:SJ
- moved J3 63.8 mm to (95.2, 11.4)
Connections:
- removed net N$75: LED10.A, RL3.1
- new net N$11: IC4.26, R35.2
- new net N$29: C35.1, IC4.23
- new net N$3: IC4.18, JP3.4
- new net N$30: C34.2, IC4.22
- new net N$35: C29.1, IC4.20
- new net N$36: C31.1, IC4.1, R38.2
- new net N$40: C30.1, IC4.14, R26.2
- new net N$44: C28.1, IC4.5, R2.1, R37.2
- new net N$45: C25.1, IC4.6, R25.2
- new net N$46: C26.1, IC4.9, R27.2
- new net N$47: IC4.27, R34.1
- new net N$48: IC4.17, R7.1
- new net N$49: C27.1, IC4.8, R1.1, R28.2
- new net N$5: IC4.25, JP3.2
- new net N$51: IC4.12, R5.1, SJ7.2
- new net N$53: IC4.13, R6.1, SJ8.2
- new net N$54: IC4.16, R36.2
- new net N$55: IC4.4, JP3.1
- new net N$56: IC4.11, JP3.3
- new net N$9: C35.2, IC4.24
- net +12V: now also C33.1, C34.1, C47.+, IC4.15, IC4.28; no longer RL3.2, U$6.+12V
- net +5V: now also C32.1, IC4.10, R1.2, R2.2, R34.2, R5.2, R6.2, R7.2; no longer U$6.+5V
- net D8*: now also IC4.3
- net D9*: now also IC4.19
- net GND: now also C25.2, C26.2, C27.2, C28.2, C29.2, C30.2, C31.2, C32.2, C33.2, C47.-, IC4.21, IC4.7, IC4.P$1, R25.1, R26.1, R27.1, R28.1, R35.1, R36.1, R37.1, R38.1, SJ7.1, SJ8.1; no longer LED10.C, Q13.3, Q3.3, Q5.3, Q6.3, U$6.GND1, U$6.GND2
- net MISO: no longer Q3.1, Q5.1
- net SCK: no longer Q13.1, Q6.1

Commit message: Update eagle
Parts:
- removed RGB-J2: RJ12, lpatiny:RJ12-STRAIGHT-RGB
- added RGB_7-8-13: (no value), lpatiny:LED-TRICOLOR-THROUGHHOLE
- added RL13, RL2, RL8: 1K, resistor:M1206
- I2C-J1: value RJ12STRAIGHT-I2C -> RJ12RIGHTANGLE; device lpatiny:RJ12-STRAIGHT-I2C -> lpatiny:RJ12-RIGHTANGLE
- J1, J2, J3: device lpatiny:RJ12-STRAIGHT -> lpatiny:RJ12-RIGHTANGLE
- RGB-J1: device lpatiny:RJ12-STRAIGHT-RGB -> lpatiny:RJ12-RIGHTANGLE
- moved J2 66.7 mm to (82.5, 11.4)
- moved CON1 60.4 mm to (32.4, 64.5)
- moved X4 35.7 mm to (7.62, 5.08), turned to 90 degrees
- moved Q9 15.7 mm to (12.7, 22.9), turned to 0 degrees
- moved J3 2.54 mm to (97.8, 11.4)
Connections:
- removed net N$10: Q11.2, RGB-J2.B
- new net +5V1: RGB_7-8-13.GND
- new net N$19: RL8.1
- new net N$21: RL13.1
- new net N$22: RGB_7-8-13.RED, RL2.2
- new net N$24: RGB_7-8-13.BLU, RL8.2
- new net N$25: RGB_7-8-13.GRN, RL13.2
- new net N$26: RL2.1
- net +12V: no longer RGB-J2.+12V
- net +5V: now also Q11.2; no longer RGB-J2.+5V
- net GND: no longer RGB-J2.GND1
- net N$20: no longer RGB-J2.R
- net N$23: no longer RGB-J2.G
- net N$50: now also RGB-J1.I/O; no longer RGB-J1.B
- net N$6: now also RGB-J1.GND2; no longer RGB-J1.G
- net N$68: now also RGB-J1.PWM; no longer RGB-J1.R
- net SCL: now also I2C-J1.PWM; no longer I2C-J1.SCL
- net SDA: now also I2C-J1.I/O; no longer I2C-J1.SDA
