File: eagle/Slave/v1.sch (EAGLE design)
At the start: 77 parts, among them CON1 SPI, IC4 DRV8811, J1 RJ12, J2 RJ12, J3 RJ12, Q1 BSP75, Q10 BSP75, Q11 BSP75, Q12 BSP75, Q2 BSP75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

Commit message: Update eagle
Parts:
- removed RGB-J2: RJ12, lpatiny:RJ12STRAIGHT-RGB
- added RGB_7-8-13: (no value), lpatiny:TOPLED-3
- added RL13, RL2, RL8: 1K, resistor:R-EU_M1206
- I2C-J1: value RJ12STRAIGHT-I2C -> RJ12RIGHTANGLE; device lpatiny:RJ12STRAIGHT-I2C -> lpatiny:RJ12RIGHTANGLE
- J1, J2, J3: device lpatiny:RJ12STRAIGHT -> lpatiny:RJ12RIGHTANGLE
- RGB-J1: device lpatiny:RJ12STRAIGHT-RGB -> lpatiny:RJ12RIGHTANGLE
Connections:
- removed net N$10: Q11.D@1, RGB-J2.3
- new net +5V1: RGB_7-8-13.A2
- new net N$19: RL8.1
- new net N$21: RL13.1
- new net N$22: RGB_7-8-13.CRED, RL2.2
- new net N$24: RGB_7-8-13.CBLUE, RL8.2
- new net N$25: RGB_7-8-13.CGREEN, RL13.2
- new net N$26: RL2.1
- net +12V: no longer RGB-J2.1
- net +5V: now also Q11.D@1; no longer RGB-J2.5
- net GND: no longer RGB-J2.6
- net N$20: no longer RGB-J2.2
- net N$23: no longer RGB-J2.4
Changed lines of the file:
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@@
 </classes>
 <parts>
-<part name="J1" library="lpatiny" deviceset="RJ12" device="STRAIGHT" value="RJ12"/>
+<part name="J1" library="lpatiny" deviceset="RJ12" device="RIGHTANGLE" value="RJ12"/>
 <part name="GND9" library="supply1" deviceset="GND" device=""/>
 <part name="R" library="rcl" deviceset="R-EU_" device="R0805" value="1k"/>
 <part name="P+8" library="supply1" deviceset="+12V" device=""/>
-<part name="J2" library="lpatiny" deviceset="RJ12" device="STRAIGHT" value="RJ12"/>
+<part name="J2" library="lpatiny" deviceset="RJ12" device="RIGHTANGLE" value="RJ12"/>
 <part name="GND6" library="supply1" deviceset="GND" device=""/>
 <part name="SUPPLY6" library="supply1" deviceset="+5V" device=""/>
 <part name="R32" library="rcl" deviceset="R-EU_" device="R0805" value="1k"/>
 <part name="P+12" library="supply1" deviceset="+12V" device=""/>
-<part name="J3" library="lpatiny" deviceset="RJ12" device="STRAIGHT" value="RJ12"/>
+<part name="J3" library="lpatiny" deviceset="RJ12" device="RIGHTANGLE" value="RJ12"/>
 <part name="GND22" library="supply1" deviceset="GND" device=""/>
 <part name="SUPPLY7" library="supply1" deviceset="+5V" device=""/>
@@
 <part name="GND13" library="supply1" deviceset="GND" device=""/>
 <part name="GND16" library="supply1" deviceset="GND" device=""/>
-<part name="RGB-J1" library="lpatiny" deviceset="RJ12" device="STRAIGHT-RGB" value="RJ12"/>
+<part name="RGB-J1" library="lpatiny" deviceset="RJ12" device="RIGHTANGLE" value="RJ12"/>
 <part name="GND5" library="supply1" deviceset="GND" device=""/>
 <part name="P+41" library="supply1" deviceset="+5V" device=""/>
@@
 <part name="GND34" library="supply1" deviceset="GND" device=""/>
 <part name="GND35" library="supply1" deviceset="GND" device=""/>
-<part name="I2C-J1" library="lpatiny" deviceset="RJ12" device="STRAIGHT-I2C" value="RJ12STRAIGHT-I2C"/>
+<part name="I2C-J1" library="lpatiny" deviceset="RJ12" device="RIGHTANGLE" value="RJ12RIGHTANGLE"/>
 <part name="R29" library="resistor" deviceset="R-EU_" device="M0805" value="10K"/>
 <part name="R30" library="resistor" deviceset="R-EU_" device="M0805" value="10K"/>
@@
 <part name="GND8" library="supply1" deviceset="GND" device=""/>
 <part name="GND27" library="supply1" deviceset="GND" device=""/>
-<part name="RGB-J2" library="lpatiny" deviceset="RJ12" device="STRAIGHT-RGB" value="RJ12"/>
 <part name="GND2" library="supply1" deviceset="GND" device=""/>
 <part name="P+2" library="supply1" deviceset="+5V" device=""/>
-<part name="P+3" library="supply1" deviceset="+12V" device=""/>
 <part name="Q7" library="infineon" deviceset="BSP613P" device="" value="BSP75"/>
 <part name="Q11" library="infineon" deviceset="BSP613P" device="" value="BSP75"/>
@@
 <part name="P+19" library="supply1" deviceset="+5V" device=""/>
 <part name="P+20" library="supply1" deviceset="+5V" device=""/>
+<part name="RL2" library="resistor" deviceset="R-EU_" device="M1206" value="1K"/>
+<part name="RL8" library="resistor" deviceset="R-EU_" device="M1206" value="1K"/>
+<part name="RL13" library="resistor" deviceset="R-EU_" device="M1206" value="1K"/>
+<part name="RGB_7-8-13" library="lpatiny" deviceset="TOPLED-3" device=""/>
+<part name="P+3" library="supply1" deviceset="+5V" device=""/>
 </parts>
 <sheets>
@@
 <instance part="GND8" gate="1" x="307.34" y="17.78"/>
 <instance part="GND27" gate="1" x="297.18" y="22.86"/>
-<instance part="RGB-J2" gate="G$1" x="375.92" y="292.1" smashed="yes" rot="R90">
-<attribute name="NAME" x="374.015" y="300.355" size="1.778" layer="95" rot="R90"/>
-</instance>
-<instance part="GND2" gate="1" x="386.08" y="287.02" smashed="yes" rot="R90">
-<attribute name="VALUE" x="387.985" y="285.115" size="1.27" layer="96" rot="R90"/>
-</instance>
-<instance part="P+2" gate="1" x="383.54" y="284.48" smashed="yes" rot="R270">
-<attribute name="VALUE" x="384.175" y="285.115" size="1.27" layer="96" rot="R90"/>
-</instance>
-<instance part="P+3" gate="1" x="368.3" y="287.02" smashed="yes" rot="R90">
-<attribute name="VALUE" x="368.3" y="288.925" size="1.27" layer="96" rot="R90"/>
+<instance part="GND2" gate="1" x="439.42" y="297.18" smashed="yes" rot="R90">
+<attribute name="VALUE" x="441.325" y="295.275" size="1.27" layer="96" rot="R90"/>
+</instance>
+<instance part="P+2" gate="1" x="447.04" y="264.16" smashed="yes" rot="R270">
+<attribute name="VALUE" x="447.675" y="264.795" size="1.27" layer="96" rot="R90"/>
 </instance>
 <instance part="Q7" gate="G$1" x="360.68" y="246.38"/>
@@
 <attribute name="VALUE" x="593.725" y="120.015" size="1.27" layer="96" rot="R180"/>
 </instance>
+<instance part="RL2" gate="G$1" x="419.1" y="264.16" smashed="yes" rot="MR180">
+<attribute name="NAME" x="417.195" y="264.5664" size="1.016" layer="95" rot="MR180"/>
+<attribute name="VALUE" x="420.37" y="264.287" size="1.016" layer="96" rot="MR180"/>
+</instance>
+<instance part="RL8" gate="G$1" x="419.1" y="259.08" smashed="yes" rot="MR180">
+<attribute name="NAME" x="417.195" y="259.4864" size="1.016" layer="95" rot="MR180"/>
+<attribute name="VALUE" x="420.37" y="259.207" size="1.016" layer="96" rot="MR180"/>
+</instance>
+<instance part="RL13" gate="G$1" x="419.1" y="254" smashed="yes" rot="MR180">
+<attribute name="NAME" x="417.195" y="254.4064" size="1.016" layer="95" rot="MR180"/>
+<attribute name="VALUE" x="420.37" y="254.127" size="1.016" layer="96" rot="MR180"/>
+</instance>
+<instance part="RGB_7-8-13" gate="G$1" x="429.26" y="259.08" rot="R270"/>
+<instance part="P+3" gate="1" x="378.46" y="289.56" smashed="yes" rot="R270">
+<attribute name="VALUE" x="379.095" y="290.195" size="1.27" layer="96" rot="R90"/>
+</instance>
 </instances>
 <busses>
@@
 </segment>
 <segment>
-<wire x1="381" y1="284.48" x2="381" y2="289.56" width="0.1524" layer="91"/>
-<pinref part="RGB-J2" gate="G$1" pin="5"/>
-<pinref part="P+2" gate="1" pin="+5V"/>
-</segment>
-<segment>
 <pinref part="R1" gate="G$1" pin="2"/>
 <wire x1="452.12" y1="114.3" x2="452.12" y2="111.76" width="0.1524" layer="91"/>
@@
 <pinref part="P+10" gate="1" pin="+5V"/>
 <junction x="472.44" y="114.3"/>
+</segment>
+<segment>
+<pinref part="Q11" gate="G$1" pin="D@1"/>
+<wire x1="375.92" y1="289.56" x2="375.92" y2="251.46" width="0.1524" layer="91"/>
+<junction x="375.92" y="251.46"/>
+<pinref part="P+3" gate="1" pin="+5V"/>
 </segment>
 </net>
@@
 </segment>
 <segment>
-<wire x1="383.54" y1="287.02" x2="383.54" y2="289.56" width="0.1524" layer="91"/>
-<pinref part="GND2" gate="1" pin="GND"/>
-<pinref part="RGB-J2" gate="G$1" pin="6"/>
-</segment>
-<segment>
 <pinref part="Q7" gate="G$1" pin="S"/>
 <pinref part="GND3" gate="1" pin="GND"/>
@@
 <wire x1="312.42" y1="33.02" x2="292.1" y2="33.02" width="0.1524" layer="91"/>
 <label x="295.402" y="33.782" size="1.778" layer="95"/>
-</segment>
-<segment>
-<wire x1="370.84" y1="289.56" x2="370.84" y2="287.02" width="0.1524" layer="91"/>
-<pinref part="RGB-J2" gate="G$1" pin="1"/>
-<pinref part="P+3" gate="1" pin="+12V"/>
 </segment>
 <segment>
@@
 </segment>
 </net>
-<net name="N$10" class="4">
-<segment>
-<pinref part="RGB-J2" gate="G$1" pin="3"/>
-<pinref part="Q11" gate="G$1" pin="D@1"/>
-<wire x1="375.92" y1="289.56" x2="375.92" y2="251.46" width="0.1524" layer="91"/>
-<junction x="375.92" y="251.46"/>
-</segment>
-</net>
 <net name="N$20" class="4">
 <segment>
-<pinref part="RGB-J2" gate="G$1" pin="2"/>
-<wire x1="373.38" y1="259.08" x2="373.38" y2="289.56" width="0.1524" layer="91"/>
 <pinref part="Q7" gate="G$1" pin="D@1"/>
-<wire x1="373.38" y1="259.08" x2="363.22" y2="259.08" width="0.1524" layer="91"/>
 <wire x1="363.22" y1="259.08" x2="363.22" y2="251.46" width="0.1524" layer="91"/>
 <junction x="363.22" y="251.46"/>
@@
 <net name="N$23" class="4">
 <segment>
-<pinref part="RGB-J2" gate="G$1" pin="4"/>
 <pinref part="Q12" gate="G$1" pin="D@1"/>
-<wire x1="378.46" y1="259.08" x2="378.46" y2="289.56" width="0.1524" layer="91"/>
-<wire x1="378.46" y1="259.08" x2="388.62" y2="259.08" width="0.1524" layer="91"/>
 <wire x1="388.62" y1="259.08" x2="388.62" y2="251.46" width="0.1524" layer="91"/>
 <junction x="388.62" y="251.46"/>
@@
 </segment>
 </net>
+<net name="+5V1" class="2">
+<segment>
+<wire x1="434.34" y1="264.16" x2="444.5" y2="264.16" width="0.1524" layer="91"/>
+<pinref part="RGB_7-8-13" gate="G$1" pin="A2"/>
+<pinref part="P+2" gate="1" pin="+5V"/>
+</segment>
+</net>
+<net name="N$19" class="1">
+<segment>
+<wire x1="414.02" y1="259.08" x2="396.24" y2="259.08" width="0.1524" layer="91"/>
+<pinref part="RL8" gate="G$1" pin="1"/>
+</segment>
+</net>
+<net name="N$21" class="1">
+<segment>
+<wire x1="414.02" y1="254" x2="403.86" y2="254" width="0.1524" layer="91"/>
+<pinref part="RL13" gate="G$1" pin="1"/>
+</segment>
+</net>
+<net name="N$22" class="0">
+<segment>
+<wire x1="426.72" y1="264.16" x2="424.18" y2="264.16" width="0.1524" layer="91"/>
+<pinref part="RGB_7-8-13" gate="G$1" pin="CRED"/>
+<pinref part="RL2" gate="G$1" pin="2"/>
+</segment>
+</net>
+<net name="N$24" class="0">
+<segment>
+<wire x1="426.72" y1="259.08" x2="424.18" y2="259.08" width="0.1524" layer="91"/>
+<pinref part="RGB_7-8-13" gate="G$1" pin="CBLUE"/>
+<pinref part="RL8" gate="G$1" pin="2"/>
+</segment>
+</net>
+<net name="N$25" class="0">
+<segment>
+<wire x1="426.72" y1="254" x2="424.18" y2="254" width="0.1524" layer="91"/>
+<pinref part="RGB_7-8-13" gate="G$1" pin="CGREEN"/>
+<pinref part="RL13" gate="G$1" pin="2"/>
+</segment>
+</net>
+<net name="N$26" class="1">
+<segment>
+<wire x1="414.02" y1="264.16" x2="403.86" y2="264.16" width="0.1524" layer="91"/>
+<pinref part="RL2" gate="G$1" pin="1"/>
+</segment>
+</net>
